File: 1.KiCADFiles/Single.Channel/Single.Channel.Amp.kicad_pcb (KiCad board)
At the start: 2 copper layers, 50 x 43.8 mm, 20 parts

Commit message: Updated Single Channel Test Board, Generated Gerber and Plot Files
Parts:
- removed the ? at (38.2, 58.1)
- removed the ? at (61.2, 58.1)
- added REF**: SMA_Amphenol_901-144_Vertical, Connector_Coaxial:SMA_Amphenol_901-144_Vertical, F.Cu at (38.2, 59.1)
- added REF**: SMA_Amphenol_901-144_Vertical, Connector_Coaxial:SMA_Amphenol_901-144_Vertical, F.Cu at (61.2, 59.1)
Routing:
- net (no net): track 67.5 -> 69.5 mm
Other:
- board text added: "In"
- board text added: "Out"
- board text removed: "Input"
- board text removed: "Output"
