File: 1.KiCADFiles/Single.Channel.v2/Single.Channel.Amp.kicad_sch (KiCad schematic)
At the start: 18 parts, among them J2 Conn_01x08, J3 Conn_01x04, J4 Conn_Coaxial_In, J5 Conn_Coaxial_Out, Q1 MMBT3904, Q2 MMBT3906

Commit message: Updated Voltage Reference Points
Connections:
- net GND: now also C3.2, C4.2; no longer J4.2 (Ext), J5.2 (Ext)
- net GND1: now also J4.2 (Ext), J5.2 (Ext); no longer C3.2, C4.2
Other:
- moved on the sheet: J2, J4, J5
