File: 1.KiCADFiles/32.Channel.Amp/32.Channel.Amp.kicad_pcb (KiCad board)
At the start: 4 copper layers, 195.8 x 139 mm, 24 parts, among them J4 Conn_01x08, Q1 MMBT3904, Q2 MMBT3906

Commit message: Updated Preview Files, Added Cell Pin Blueprint, Created Cell Tester
Parts:
- removed the REF** at (137.6, 117.5)
- removed the REF** at (137.6, 82.5)
- added G***: LOGO, 1.Logos:UTA, F.Cu at (200.0, 154.0)
- added G***: LOGO, 1.Logos:UTA, F.Cu at (123.1, 107.6)
- added J5: Conn_Coaxial_Out, Connector_Coaxial:SMA_Amphenol_901-144_Vertical, F.Cu at (120.0, 74.8)
- added J5: Conn_Coaxial_Out, Connector_Coaxial:SMA_Amphenol_901-144_Vertical, F.Cu at (120.0, 124.8)
- added REF**: DSUB-9_Female_Horizontal_P2.77x2.54mm_EdgePinOffset9.40mm, Connector_Dsub:DSUB-9_Female_Horizontal_P2.77x2.54mm_EdgePinOffset9.40mm, F.Cu at (107.5, 105.3)
- moved C4 55.4 mm to (35.1, 106.6)
- moved D1 55.4 mm to (26.1, 91.7)
- moved D3 55.4 mm to (30.4, 96.1)
- moved D4 55.4 mm to (36.5, 110.7)
- moved Q1 55.4 mm to (25.4, 100.8)
- moved Q2 55.4 mm to (34.2, 105.9)
- moved R2 55.4 mm to (35.7, 101.7)
- moved C2 55.4 mm to (35.8, 98.8)
- moved D2 55.4 mm to (35.3, 96.2)
- moved R4 55.4 mm to (33.5, 111.1)
- moved REF** 55.4 mm to (39.0, 122.1)
- moved REF** 55.4 mm to (39.0, 92.6)
- moved REF** 55.4 mm to (39.0, 89.6)
- moved REF** 55.4 mm to (39.0, 124.6)
- moved C1 55.4 mm to (26.0, 94.8)
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Other:
- board size 195.8 x 139 mm -> 251 x 142 mm
- board text added: "32 Cell Receiver Board July 2023 Alfredo Barajas Enriquez"
- board text added: ":: Board Details :: Layers: 4 Dimensions: 142 x 142 mm"
- board text added: "Cell Tester July 2023 Alfredo Barajas Enriquez"
- board text removed: "32 Cell Receivver Board July 2023 Alfredo Barajas Enriquez"
