File: 1.KiCADFiles/Receiver.Board/Receiver.Board.kicad_pcb (KiCad board)
At the start: 4 copper layers, 251 x 142 mm, 27 parts, among them J4 Conn_01x08, J5 Conn_Coaxial_Out, Q1 MMBT3904, Q2 MMBT3906

Commit message: Cleaned Files
Other:
- board text added: "32 Cell Receiver Board v.1 July 2023 Alfredo Barajas Enriquez"
- board text removed: "32 Cell Receiver Board July 2023 Alfredo Barajas Enriquez"
Changed lines of the file:
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@@
     (effects (font (size 1.5 1.5) (thickness 0.3) bold) (justify left bottom))
   )
-  (gr_text "32 Cell Receiver Board\nJuly 2023\nAlfredo Barajas Enriquez" (at 202 150 90) (layer "F.SilkS")
+  (gr_text "32 Cell Receiver Board v.1\nJuly 2023\nAlfredo Barajas Enriquez" (at 202 150 90) (layer "F.SilkS")
     (effects (font (size 1 1) (thickness 0.15)) (justify left bottom))
   )
