File: 1.KiCADFiles/ReceiverBoard/ReceiverBoard.v2/12.Layer.receiverBoard/12.Layer.ReceiverBoard.kicad_pcb (KiCad board)
At the start: 12 copper layers, 180 x 167 mm, 2 parts

Commit message: Added Base
Parts:
- added REF**: CONN D-SUB PLUG 50POS RA SLDR, 1.Local.Library:CONN D-SUB PLUG 50POS RA SLDR, F.Cu at (75.0, 173.0)
Routing:
- net (no net): track 0.00 -> 3330.3 mm, vias 0 -> 64
- added copper zone on In11.Cu, net Power.Ground
- added copper zone on In10.Cu, net Signal.Ground
- removed copper zone on In9.Cu, net Power.Ground
Other:
- copper layers 12 -> 14
