File: 1.KiCADFiles/ReceiverBoard/ReceiverBoard.v3/8.Layer.Receiver.No.Wrap/8.Layer.Receiver.No.Wrap.kicad_pcb (KiCad board)
At the start: 8 copper layers, 180 x 167 mm, 4 parts

Commit message: Major Design Changes
Parts:
- added REF**: PinSocket_1x03_P2.54mm_Vertical, Connector_PinSocket_2.54mm:PinSocket_1x03_P2.54mm_Vertical, F.Cu at (43.0, 57.5)
- added REF**: MountingHole_4mm, MountingHole:MountingHole_4mm, B.Cu at (37.4, 155.6)
- added REF**: MountingHole_4mm, MountingHole:MountingHole_4mm, B.Cu at (202.6, 30.4)
- added REF**: MountingHole_4mm, MountingHole:MountingHole_4mm, F.Cu at (37.4, 30.4)
- added REF**: PinSocket_1x02_P2.54mm_Vertical_SMD_Pin1Right, Connector_PinSocket_2.54mm:PinSocket_1x02_P2.54mm_Vertical_SMD_Pin1Right, F.Cu at (43.0, 42.8)
- added REF**: PinSocket_1x02_P2.54mm_Vertical_SMD_Pin1Right, Connector_PinSocket_2.54mm:PinSocket_1x02_P2.54mm_Vertical_SMD_Pin1Right, F.Cu at (43.0, 75.0)
- added REF**: MountingHole_4mm, MountingHole:MountingHole_4mm, F.Cu at (120.0, 120.0)
- added REF**: MountingHole_4mm, MountingHole:MountingHole_4mm, B.Cu at (202.6, 155.6)
- added REF**1: PinSocket_1x02_P2.54mm_Vertical_SMD_Pin1Right, Connector_PinSocket_2.54mm:PinSocket_1x02_P2.54mm_Vertical_SMD_Pin1Right, F.Cu at (38.0, 115.0)
- added REF**10: PinSocket_1x02_P2.54mm_Vertical_SMD_Pin1Right, Connector_PinSocket_2.54mm:PinSocket_1x02_P2.54mm_Vertical_SMD_Pin1Right, F.Cu at (63.0, 75.0)
- added REF**11: PinSocket_1x03_P2.54mm_Vertical, Connector_PinSocket_2.54mm:PinSocket_1x03_P2.54mm_Vertical, F.Cu at (63.0, 57.5)
- added REF**12: PinSocket_1x02_P2.54mm_Vertical_SMD_Pin1Right, Connector_PinSocket_2.54mm:PinSocket_1x02_P2.54mm_Vertical_SMD_Pin1Right, F.Cu at (63.0, 42.8)
- added REF**13: PinSocket_1x02_P2.54mm_Vertical_SMD_Pin1Right, Connector_PinSocket_2.54mm:PinSocket_1x02_P2.54mm_Vertical_SMD_Pin1Right, F.Cu at (58.0, 115.0)
- added REF**14: PinSocket_1x03_P2.54mm_Vertical, Connector_PinSocket_2.54mm:PinSocket_1x03_P2.54mm_Vertical, F.Cu at (58.0, 97.5)
- added REF**15: PinSocket_1x02_P2.54mm_Vertical_SMD_Pin1Right, Connector_PinSocket_2.54mm:PinSocket_1x02_P2.54mm_Vertical_SMD_Pin1Right, F.Cu at (58.0, 82.8)
- added REF**16: PinSocket_1x02_P2.54mm_Vertical_SMD_Pin1Right, Connector_PinSocket_2.54mm:PinSocket_1x02_P2.54mm_Vertical_SMD_Pin1Right, F.Cu at (73.0, 75.0)
- added REF**17: PinSocket_1x03_P2.54mm_Vertical, Connector_PinSocket_2.54mm:PinSocket_1x03_P2.54mm_Vertical, F.Cu at (73.0, 57.5)
- added REF**18: PinSocket_1x02_P2.54mm_Vertical_SMD_Pin1Right, Connector_PinSocket_2.54mm:PinSocket_1x02_P2.54mm_Vertical_SMD_Pin1Right, F.Cu at (73.0, 42.8)
- added REF**19: PinSocket_1x02_P2.54mm_Vertical_SMD_Pin1Right, Connector_PinSocket_2.54mm:PinSocket_1x02_P2.54mm_Vertical_SMD_Pin1Right, F.Cu at (68.0, 115.0)
- added REF**2: PinSocket_1x03_P2.54mm_Vertical, Connector_PinSocket_2.54mm:PinSocket_1x03_P2.54mm_Vertical, F.Cu at (38.0, 97.5)
- added REF**20: PinSocket_1x03_P2.54mm_Vertical, Connector_PinSocket_2.54mm:PinSocket_1x03_P2.54mm_Vertical, F.Cu at (68.0, 97.5)
- added REF**21: PinSocket_1x02_P2.54mm_Vertical_SMD_Pin1Right, Connector_PinSocket_2.54mm:PinSocket_1x02_P2.54mm_Vertical_SMD_Pin1Right, F.Cu at (68.0, 82.8)
- added REF**22: PinSocket_1x02_P2.54mm_Vertical_SMD_Pin1Right, Connector_PinSocket_2.54mm:PinSocket_1x02_P2.54mm_Vertical_SMD_Pin1Right, F.Cu at (83.0, 75.0)
- added REF**23: PinSocket_1x03_P2.54mm_Vertical, Connector_PinSocket_2.54mm:PinSocket_1x03_P2.54mm_Vertical, F.Cu at (83.0, 57.5)
- added REF**24: PinSocket_1x02_P2.54mm_Vertical_SMD_Pin1Right, Connector_PinSocket_2.54mm:PinSocket_1x02_P2.54mm_Vertical_SMD_Pin1Right, F.Cu at (83.0, 42.8)
- added REF**25: PinSocket_1x02_P2.54mm_Vertical_SMD_Pin1Right, Connector_PinSocket_2.54mm:PinSocket_1x02_P2.54mm_Vertical_SMD_Pin1Right, F.Cu at (78.0, 115.0)
- added REF**26: PinSocket_1x03_P2.54mm_Vertical, Connector_PinSocket_2.54mm:PinSocket_1x03_P2.54mm_Vertical, F.Cu at (78.0, 97.5)
- added REF**27: PinSocket_1x02_P2.54mm_Vertical_SMD_Pin1Right, Connector_PinSocket_2.54mm:PinSocket_1x02_P2.54mm_Vertical_SMD_Pin1Right, F.Cu at (78.0, 82.8)
- added REF**28: PinSocket_1x02_P2.54mm_Vertical_SMD_Pin1Right, Connector_PinSocket_2.54mm:PinSocket_1x02_P2.54mm_Vertical_SMD_Pin1Right, F.Cu at (93.0, 75.0)
- added REF**29: PinSocket_1x03_P2.54mm_Vertical, Connector_PinSocket_2.54mm:PinSocket_1x03_P2.54mm_Vertical, F.Cu at (93.0, 57.5)
- added REF**3: PinSocket_1x02_P2.54mm_Vertical_SMD_Pin1Right, Connector_PinSocket_2.54mm:PinSocket_1x02_P2.54mm_Vertical_SMD_Pin1Right, F.Cu at (38.0, 82.8)
- added REF**30: PinSocket_1x02_P2.54mm_Vertical_SMD_Pin1Right, Connector_PinSocket_2.54mm:PinSocket_1x02_P2.54mm_Vertical_SMD_Pin1Right, F.Cu at (93.0, 42.8)
- added REF**31: PinSocket_1x02_P2.54mm_Vertical_SMD_Pin1Right, Connector_PinSocket_2.54mm:PinSocket_1x02_P2.54mm_Vertical_SMD_Pin1Right, F.Cu at (88.0, 115.0)
- added REF**32: PinSocket_1x03_P2.54mm_Vertical, Connector_PinSocket_2.54mm:PinSocket_1x03_P2.54mm_Vertical, F.Cu at (88.0, 97.5)
- added REF**33: PinSocket_1x02_P2.54mm_Vertical_SMD_Pin1Right, Connector_PinSocket_2.54mm:PinSocket_1x02_P2.54mm_Vertical_SMD_Pin1Right, F.Cu at (88.0, 82.8)
- added REF**34: PinSocket_1x02_P2.54mm_Vertical_SMD_Pin1Right, Connector_PinSocket_2.54mm:PinSocket_1x02_P2.54mm_Vertical_SMD_Pin1Right, F.Cu at (103.0, 75.0)
- added REF**35: PinSocket_1x03_P2.54mm_Vertical, Connector_PinSocket_2.54mm:PinSocket_1x03_P2.54mm_Vertical, F.Cu at (103.0, 57.5)
- added REF**36: PinSocket_1x02_P2.54mm_Vertical_SMD_Pin1Right, Connector_PinSocket_2.54mm:PinSocket_1x02_P2.54mm_Vertical_SMD_Pin1Right, F.Cu at (103.0, 42.8)
- added REF**37: PinSocket_1x02_P2.54mm_Vertical_SMD_Pin1Right, Connector_PinSocket_2.54mm:PinSocket_1x02_P2.54mm_Vertical_SMD_Pin1Right, F.Cu at (98.0, 115.0)
- added REF**38: PinSocket_1x03_P2.54mm_Vertical, Connector_PinSocket_2.54mm:PinSocket_1x03_P2.54mm_Vertical, F.Cu at (98.0, 97.5)
- added REF**39: PinSocket_1x02_P2.54mm_Vertical_SMD_Pin1Right, Connector_PinSocket_2.54mm:PinSocket_1x02_P2.54mm_Vertical_SMD_Pin1Right, F.Cu at (98.0, 82.8)
- added REF**4: PinSocket_1x02_P2.54mm_Vertical_SMD_Pin1Right, Connector_PinSocket_2.54mm:PinSocket_1x02_P2.54mm_Vertical_SMD_Pin1Right, F.Cu at (53.0, 75.0)
- added REF**40: PinSocket_1x02_P2.54mm_Vertical_SMD_Pin1Right, Connector_PinSocket_2.54mm:PinSocket_1x02_P2.54mm_Vertical_SMD_Pin1Right, F.Cu at (113.0, 75.0)
- added REF**41: PinSocket_1x03_P2.54mm_Vertical, Connector_PinSocket_2.54mm:PinSocket_1x03_P2.54mm_Vertical, F.Cu at (113.0, 57.5)
- added REF**42: PinSocket_1x02_P2.54mm_Vertical_SMD_Pin1Right, Connector_PinSocket_2.54mm:PinSocket_1x02_P2.54mm_Vertical_SMD_Pin1Right, F.Cu at (113.0, 42.8)
- added REF**43: PinSocket_1x02_P2.54mm_Vertical_SMD_Pin1Right, Connector_PinSocket_2.54mm:PinSocket_1x02_P2.54mm_Vertical_SMD_Pin1Right, F.Cu at (108.0, 115.0)
- added REF**44: PinSocket_1x03_P2.54mm_Vertical, Connector_PinSocket_2.54mm:PinSocket_1x03_P2.54mm_Vertical, F.Cu at (108.0, 97.5)
- added REF**45: PinSocket_1x02_P2.54mm_Vertical_SMD_Pin1Right, Connector_PinSocket_2.54mm:PinSocket_1x02_P2.54mm_Vertical_SMD_Pin1Right, F.Cu at (108.0, 82.8)
- added REF**46: PinSocket_1x02_P2.54mm_Vertical_SMD_Pin1Right, Connector_PinSocket_2.54mm:PinSocket_1x02_P2.54mm_Vertical_SMD_Pin1Right, F.Cu at (123.0, 75.0)
- added REF**47: PinSocket_1x03_P2.54mm_Vertical, Connector_PinSocket_2.54mm:PinSocket_1x03_P2.54mm_Vertical, F.Cu at (123.0, 57.5)
- added REF**48: PinSocket_1x02_P2.54mm_Vertical_SMD_Pin1Right, Connector_PinSocket_2.54mm:PinSocket_1x02_P2.54mm_Vertical_SMD_Pin1Right, F.Cu at (123.0, 42.8)
- added REF**5: PinSocket_1x03_P2.54mm_Vertical, Connector_PinSocket_2.54mm:PinSocket_1x03_P2.54mm_Vertical, F.Cu at (53.0, 57.5)
- added REF**52: PinSocket_1x02_P2.54mm_Vertical_SMD_Pin1Right, Connector_PinSocket_2.54mm:PinSocket_1x02_P2.54mm_Vertical_SMD_Pin1Right, F.Cu at (133.0, 75.0)
- added REF**53: PinSocket_1x03_P2.54mm_Vertical, Connector_PinSocket_2.54mm:PinSocket_1x03_P2.54mm_Vertical, F.Cu at (133.0, 57.5)
- added REF**54: PinSocket_1x02_P2.54mm_Vertical_SMD_Pin1Right, Connector_PinSocket_2.54mm:PinSocket_1x02_P2.54mm_Vertical_SMD_Pin1Right, F.Cu at (133.0, 42.8)
- added REF**55: PinSocket_1x02_P2.54mm_Vertical_SMD_Pin1Right, Connector_PinSocket_2.54mm:PinSocket_1x02_P2.54mm_Vertical_SMD_Pin1Right, F.Cu at (128.0, 115.0)
- added REF**56: PinSocket_1x03_P2.54mm_Vertical, Connector_PinSocket_2.54mm:PinSocket_1x03_P2.54mm_Vertical, F.Cu at (128.0, 97.5)
- added REF**57: PinSocket_1x02_P2.54mm_Vertical_SMD_Pin1Right, Connector_PinSocket_2.54mm:PinSocket_1x02_P2.54mm_Vertical_SMD_Pin1Right, F.Cu at (128.0, 82.8)
- added REF**58: PinSocket_1x02_P2.54mm_Vertical_SMD_Pin1Right, Connector_PinSocket_2.54mm:PinSocket_1x02_P2.54mm_Vertical_SMD_Pin1Right, F.Cu at (143.0, 75.0)
- added REF**59: PinSocket_1x03_P2.54mm_Vertical, Connector_PinSocket_2.54mm:PinSocket_1x03_P2.54mm_Vertical, F.Cu at (143.0, 57.5)
- added REF**6: PinSocket_1x02_P2.54mm_Vertical_SMD_Pin1Right, Connector_PinSocket_2.54mm:PinSocket_1x02_P2.54mm_Vertical_SMD_Pin1Right, F.Cu at (53.0, 42.8)
- added REF**60: PinSocket_1x02_P2.54mm_Vertical_SMD_Pin1Right, Connector_PinSocket_2.54mm:PinSocket_1x02_P2.54mm_Vertical_SMD_Pin1Right, F.Cu at (143.0, 42.8)
- added REF**61: PinSocket_1x02_P2.54mm_Vertical_SMD_Pin1Right, Connector_PinSocket_2.54mm:PinSocket_1x02_P2.54mm_Vertical_SMD_Pin1Right, F.Cu at (138.0, 115.0)
- added REF**62: PinSocket_1x03_P2.54mm_Vertical, Connector_PinSocket_2.54mm:PinSocket_1x03_P2.54mm_Vertical, F.Cu at (138.0, 97.5)
- added REF**63: PinSocket_1x02_P2.54mm_Vertical_SMD_Pin1Right, Connector_PinSocket_2.54mm:PinSocket_1x02_P2.54mm_Vertical_SMD_Pin1Right, F.Cu at (138.0, 82.8)
- added REF**64: PinSocket_1x02_P2.54mm_Vertical_SMD_Pin1Right, Connector_PinSocket_2.54mm:PinSocket_1x02_P2.54mm_Vertical_SMD_Pin1Right, F.Cu at (153.0, 75.0)
- added REF**65: PinSocket_1x03_P2.54mm_Vertical, Connector_PinSocket_2.54mm:PinSocket_1x03_P2.54mm_Vertical, F.Cu at (153.0, 57.5)
- added REF**66: PinSocket_1x02_P2.54mm_Vertical_SMD_Pin1Right, Connector_PinSocket_2.54mm:PinSocket_1x02_P2.54mm_Vertical_SMD_Pin1Right, F.Cu at (153.0, 42.8)
- added REF**67: PinSocket_1x02_P2.54mm_Vertical_SMD_Pin1Right, Connector_PinSocket_2.54mm:PinSocket_1x02_P2.54mm_Vertical_SMD_Pin1Right, F.Cu at (148.0, 115.0)
- added REF**68: PinSocket_1x03_P2.54mm_Vertical, Connector_PinSocket_2.54mm:PinSocket_1x03_P2.54mm_Vertical, F.Cu at (148.0, 97.5)
- added REF**69: PinSocket_1x02_P2.54mm_Vertical_SMD_Pin1Right, Connector_PinSocket_2.54mm:PinSocket_1x02_P2.54mm_Vertical_SMD_Pin1Right, F.Cu at (148.0, 82.8)
- added REF**7: PinSocket_1x02_P2.54mm_Vertical_SMD_Pin1Right, Connector_PinSocket_2.54mm:PinSocket_1x02_P2.54mm_Vertical_SMD_Pin1Right, F.Cu at (48.0, 115.0)
- added REF**70: PinSocket_1x02_P2.54mm_Vertical_SMD_Pin1Right, Connector_PinSocket_2.54mm:PinSocket_1x02_P2.54mm_Vertical_SMD_Pin1Right, F.Cu at (163.0, 75.0)
- added REF**71: PinSocket_1x03_P2.54mm_Vertical, Connector_PinSocket_2.54mm:PinSocket_1x03_P2.54mm_Vertical, F.Cu at (163.0, 57.5)
- added REF**72: PinSocket_1x02_P2.54mm_Vertical_SMD_Pin1Right, Connector_PinSocket_2.54mm:PinSocket_1x02_P2.54mm_Vertical_SMD_Pin1Right, F.Cu at (163.0, 42.8)
- added REF**73: PinSocket_1x02_P2.54mm_Vertical_SMD_Pin1Right, Connector_PinSocket_2.54mm:PinSocket_1x02_P2.54mm_Vertical_SMD_Pin1Right, F.Cu at (158.0, 115.0)
- added REF**74: PinSocket_1x03_P2.54mm_Vertical, Connector_PinSocket_2.54mm:PinSocket_1x03_P2.54mm_Vertical, F.Cu at (158.0, 97.5)
- added REF**75: PinSocket_1x02_P2.54mm_Vertical_SMD_Pin1Right, Connector_PinSocket_2.54mm:PinSocket_1x02_P2.54mm_Vertical_SMD_Pin1Right, F.Cu at (158.0, 82.8)
- added REF**76: PinSocket_1x02_P2.54mm_Vertical_SMD_Pin1Right, Connector_PinSocket_2.54mm:PinSocket_1x02_P2.54mm_Vertical_SMD_Pin1Right, F.Cu at (173.0, 75.0)
- added REF**77: PinSocket_1x03_P2.54mm_Vertical, Connector_PinSocket_2.54mm:PinSocket_1x03_P2.54mm_Vertical, F.Cu at (173.0, 57.5)
- added REF**78: PinSocket_1x02_P2.54mm_Vertical_SMD_Pin1Right, Connector_PinSocket_2.54mm:PinSocket_1x02_P2.54mm_Vertical_SMD_Pin1Right, F.Cu at (173.0, 42.8)
- added REF**79: PinSocket_1x02_P2.54mm_Vertical_SMD_Pin1Right, Connector_PinSocket_2.54mm:PinSocket_1x02_P2.54mm_Vertical_SMD_Pin1Right, F.Cu at (168.0, 115.0)
- added REF**8: PinSocket_1x03_P2.54mm_Vertical, Connector_PinSocket_2.54mm:PinSocket_1x03_P2.54mm_Vertical, F.Cu at (48.0, 97.5)
- added REF**80: PinSocket_1x03_P2.54mm_Vertical, Connector_PinSocket_2.54mm:PinSocket_1x03_P2.54mm_Vertical, F.Cu at (168.0, 97.5)
- added REF**81: PinSocket_1x02_P2.54mm_Vertical_SMD_Pin1Right, Connector_PinSocket_2.54mm:PinSocket_1x02_P2.54mm_Vertical_SMD_Pin1Right, F.Cu at (168.0, 82.8)
- added REF**82: PinSocket_1x02_P2.54mm_Vertical_SMD_Pin1Right, Connector_PinSocket_2.54mm:PinSocket_1x02_P2.54mm_Vertical_SMD_Pin1Right, F.Cu at (183.0, 75.0)
- added REF**83: PinSocket_1x03_P2.54mm_Vertical, Connector_PinSocket_2.54mm:PinSocket_1x03_P2.54mm_Vertical, F.Cu at (183.0, 57.5)
- added REF**84: PinSocket_1x02_P2.54mm_Vertical_SMD_Pin1Right, Connector_PinSocket_2.54mm:PinSocket_1x02_P2.54mm_Vertical_SMD_Pin1Right, F.Cu at (183.0, 42.8)
- added REF**85: PinSocket_1x02_P2.54mm_Vertical_SMD_Pin1Right, Connector_PinSocket_2.54mm:PinSocket_1x02_P2.54mm_Vertical_SMD_Pin1Right, F.Cu at (178.0, 115.0)
- added REF**86: PinSocket_1x03_P2.54mm_Vertical, Connector_PinSocket_2.54mm:PinSocket_1x03_P2.54mm_Vertical, F.Cu at (178.0, 97.5)
- added REF**87: PinSocket_1x02_P2.54mm_Vertical_SMD_Pin1Right, Connector_PinSocket_2.54mm:PinSocket_1x02_P2.54mm_Vertical_SMD_Pin1Right, F.Cu at (178.0, 82.8)
- added REF**88: PinSocket_1x02_P2.54mm_Vertical_SMD_Pin1Right, Connector_PinSocket_2.54mm:PinSocket_1x02_P2.54mm_Vertical_SMD_Pin1Right, F.Cu at (193.0, 75.0)
- added REF**89: PinSocket_1x03_P2.54mm_Vertical, Connector_PinSocket_2.54mm:PinSocket_1x03_P2.54mm_Vertical, F.Cu at (193.0, 57.5)
- added REF**9: PinSocket_1x02_P2.54mm_Vertical_SMD_Pin1Right, Connector_PinSocket_2.54mm:PinSocket_1x02_P2.54mm_Vertical_SMD_Pin1Right, F.Cu at (48.0, 82.8)
- added REF**90: PinSocket_1x02_P2.54mm_Vertical_SMD_Pin1Right, Connector_PinSocket_2.54mm:PinSocket_1x02_P2.54mm_Vertical_SMD_Pin1Right, F.Cu at (193.0, 42.8)
- added REF**91: PinSocket_1x02_P2.54mm_Vertical_SMD_Pin1Right, Connector_PinSocket_2.54mm:PinSocket_1x02_P2.54mm_Vertical_SMD_Pin1Right, F.Cu at (188.0, 115.0)
- added REF**92: PinSocket_1x03_P2.54mm_Vertical, Connector_PinSocket_2.54mm:PinSocket_1x03_P2.54mm_Vertical, F.Cu at (188.0, 97.5)
- added REF**93: PinSocket_1x02_P2.54mm_Vertical_SMD_Pin1Right, Connector_PinSocket_2.54mm:PinSocket_1x02_P2.54mm_Vertical_SMD_Pin1Right, F.Cu at (188.0, 82.8)
- added REF**97: PinSocket_1x02_P2.54mm_Vertical_SMD_Pin1Right, Connector_PinSocket_2.54mm:PinSocket_1x02_P2.54mm_Vertical_SMD_Pin1Right, F.Cu at (198.0, 115.0)
- added REF**98: PinSocket_1x03_P2.54mm_Vertical, Connector_PinSocket_2.54mm:PinSocket_1x03_P2.54mm_Vertical, F.Cu at (198.0, 97.5)
- added REF**99: PinSocket_1x02_P2.54mm_Vertical_SMD_Pin1Right, Connector_PinSocket_2.54mm:PinSocket_1x02_P2.54mm_Vertical_SMD_Pin1Right, F.Cu at (198.0, 82.8)
- moved REF** 48.1 mm to (120.0, 156.0)
- moved REF** 18.2 mm to (184.0, 150.0)
- moved G*** 3.00 mm to (119.6, 111.7)
Connections:
- REF** pad 17: (no net) -> Signal.Ground (x2)
- REF** pad 1: (no net) -> Signal.Ground
Routing:
- net (no net): track 3330.0 -> 2388.1 mm
- net Signal.Ground: vias 14 -> 30
Other:
- board size 180 x 167 mm -> 180 x 150 mm
- board text added: "::: Copper///FR4 Stackup ::: ■ S.GND -- 18 um □ FR4 -- 0.254 mm ■ S.Trace.1 -- 18 um □ FR4 -- 0.254 mm ■ S.GND -- 18 um □ FR4 -- 0.5 mm ■ S.GND -- 18 um □ FR4 -- 0.254 mm ■ S.Trace.2 -- 18 um □ FR4 -- 0.254 mm ■ S.GND -- 18 um □ FR4 -- 0.5 mm ■ P.GND -- 18 um □ FR4 -- 0.254 mm ■ P.Trace -- 18 um"
- board text added: "::: Other ::: ▪ Trace Impedance -- 48.268 Ohms ▪ Trace Inductance -- 3.4541 nH/cm ▪ Trace Capacitance -- 1.4826 pF/cm ▪ Trace Signal Delay -- 71.5624 ps/cm ▪ Via Impedance -- 49.263 Ohms"
- board text added: "August 2023 32 Channel Pixel Receiver Board Alfredo Barajas Enriquez"
- board text removed: "32 Channel Pixel Receiver Board August 2023 Alfredo Barajas Enriquez"
- board text removed: "::: FR4 and Copper Stackup ::: ■ S.GND -- 18 um □ FR4 -- 0.254 mm ■ S.Trace.1 -- 18 um □ FR4 -- 0.254 mm ■ S.GND -- 18 um □ FR4 -- 0.5 mm ■ S.GND -- 18 um □ FR4 -- 0.254 mm ■ S.Trace.2 -- 18 um □ FR4 -- 0.254 mm ■ S.GND -- 18 um □ FR4 -- 0.5 mm ■ P.GND -- 18 um □ FR4 -- 0.254 mm ■ P.Trace -- 18 um"
- board text removed: "::: Other ::: ▪ Input Trace Impedance -- 48.268 Ohms ▪ Input Trace Inductance -- 3.4541 nH/cm ▪ Input Trace Capacitance -- 1.4826 pF/cm ▪ Input Trace Signal Delay -- 71.5624 ps/cm"

Commit message: Updated Files
Parts:
- removed REF**81, REF**82, REF**84, REF**85: PinSocket_1x02_P2.54mm_Vertical_SMD_Pin1Right, Connector_PinSocket_2.54mm:PinSocket_1x02_P2.54mm_Vertical_SMD_Pin1Right
- removed REF**83: PinSocket_1x03_P2.54mm_Vertical, Connector_PinSocket_2.54mm:PinSocket_1x03_P2.54mm_Vertical
- added REF**: R_1206_3216Metric_Pad1.30x1.75mm_HandSolder, Resistor_SMD:R_1206_3216Metric_Pad1.30x1.75mm_HandSolder, B.Cu at (43.0, 53.0)
- added REF**: R_1206_3216Metric_Pad1.30x1.75mm_HandSolder, Resistor_SMD:R_1206_3216Metric_Pad1.30x1.75mm_HandSolder, B.Cu at (43.0, 67.0)
- added REF**100: PinSocket_1x02_P2.54mm_Vertical_SMD_Pin1Right, Connector_PinSocket_2.54mm:PinSocket_1x02_P2.54mm_Vertical_SMD_Pin1Right, F.Cu at (143.0, 42.8)
- added REF**101: PinSocket_1x02_P2.54mm_Vertical_SMD_Pin1Right, Connector_PinSocket_2.54mm:PinSocket_1x02_P2.54mm_Vertical_SMD_Pin1Right, F.Cu at (138.0, 115.0)
- added REF**102: R_1206_3216Metric_Pad1.30x1.75mm_HandSolder, Resistor_SMD:R_1206_3216Metric_Pad1.30x1.75mm_HandSolder, B.Cu at (138.0, 107.0)
- added REF**103: PinSocket_1x03_P2.54mm_Vertical, Connector_PinSocket_2.54mm:PinSocket_1x03_P2.54mm_Vertical, F.Cu at (138.0, 97.5)
- added REF**104: R_1206_3216Metric_Pad1.30x1.75mm_HandSolder, Resistor_SMD:R_1206_3216Metric_Pad1.30x1.75mm_HandSolder, B.Cu at (138.0, 93.0)
- added REF**105: PinSocket_1x02_P2.54mm_Vertical_SMD_Pin1Right, Connector_PinSocket_2.54mm:PinSocket_1x02_P2.54mm_Vertical_SMD_Pin1Right, F.Cu at (138.0, 82.8)
- added REF**106: PinSocket_1x02_P2.54mm_Vertical_SMD_Pin1Right, Connector_PinSocket_2.54mm:PinSocket_1x02_P2.54mm_Vertical_SMD_Pin1Right, F.Cu at (153.0, 75.0)
- added REF**107: R_1206_3216Metric_Pad1.30x1.75mm_HandSolder, Resistor_SMD:R_1206_3216Metric_Pad1.30x1.75mm_HandSolder, B.Cu at (153.0, 67.0)
- added REF**108: PinSocket_1x03_P2.54mm_Vertical, Connector_PinSocket_2.54mm:PinSocket_1x03_P2.54mm_Vertical, F.Cu at (153.0, 57.5)
- added REF**109: R_1206_3216Metric_Pad1.30x1.75mm_HandSolder, Resistor_SMD:R_1206_3216Metric_Pad1.30x1.75mm_HandSolder, B.Cu at (153.0, 53.0)
- added REF**110: PinSocket_1x02_P2.54mm_Vertical_SMD_Pin1Right, Connector_PinSocket_2.54mm:PinSocket_1x02_P2.54mm_Vertical_SMD_Pin1Right, F.Cu at (153.0, 42.8)
- added REF**111: PinSocket_1x02_P2.54mm_Vertical_SMD_Pin1Right, Connector_PinSocket_2.54mm:PinSocket_1x02_P2.54mm_Vertical_SMD_Pin1Right, F.Cu at (148.0, 115.0)
- added REF**112: R_1206_3216Metric_Pad1.30x1.75mm_HandSolder, Resistor_SMD:R_1206_3216Metric_Pad1.30x1.75mm_HandSolder, B.Cu at (148.0, 107.0)
- added REF**113: PinSocket_1x03_P2.54mm_Vertical, Connector_PinSocket_2.54mm:PinSocket_1x03_P2.54mm_Vertical, F.Cu at (148.0, 97.5)
- added REF**114: R_1206_3216Metric_Pad1.30x1.75mm_HandSolder, Resistor_SMD:R_1206_3216Metric_Pad1.30x1.75mm_HandSolder, B.Cu at (148.0, 93.0)
- added REF**115: PinSocket_1x02_P2.54mm_Vertical_SMD_Pin1Right, Connector_PinSocket_2.54mm:PinSocket_1x02_P2.54mm_Vertical_SMD_Pin1Right, F.Cu at (148.0, 82.8)
- added REF**116: PinSocket_1x02_P2.54mm_Vertical_SMD_Pin1Right, Connector_PinSocket_2.54mm:PinSocket_1x02_P2.54mm_Vertical_SMD_Pin1Right, F.Cu at (163.0, 75.0)
- added REF**117: R_1206_3216Metric_Pad1.30x1.75mm_HandSolder, Resistor_SMD:R_1206_3216Metric_Pad1.30x1.75mm_HandSolder, B.Cu at (163.0, 67.0)
- added REF**118: PinSocket_1x03_P2.54mm_Vertical, Connector_PinSocket_2.54mm:PinSocket_1x03_P2.54mm_Vertical, F.Cu at (163.0, 57.5)
- added REF**119: R_1206_3216Metric_Pad1.30x1.75mm_HandSolder, Resistor_SMD:R_1206_3216Metric_Pad1.30x1.75mm_HandSolder, B.Cu at (163.0, 53.0)
- added REF**120: PinSocket_1x02_P2.54mm_Vertical_SMD_Pin1Right, Connector_PinSocket_2.54mm:PinSocket_1x02_P2.54mm_Vertical_SMD_Pin1Right, F.Cu at (163.0, 42.8)
- added REF**121: PinSocket_1x02_P2.54mm_Vertical_SMD_Pin1Right, Connector_PinSocket_2.54mm:PinSocket_1x02_P2.54mm_Vertical_SMD_Pin1Right, F.Cu at (158.0, 115.0)
- added REF**122: R_1206_3216Metric_Pad1.30x1.75mm_HandSolder, Resistor_SMD:R_1206_3216Metric_Pad1.30x1.75mm_HandSolder, B.Cu at (158.0, 107.0)
- added REF**123: PinSocket_1x03_P2.54mm_Vertical, Connector_PinSocket_2.54mm:PinSocket_1x03_P2.54mm_Vertical, F.Cu at (158.0, 97.5)
- added REF**124: R_1206_3216Metric_Pad1.30x1.75mm_HandSolder, Resistor_SMD:R_1206_3216Metric_Pad1.30x1.75mm_HandSolder, B.Cu at (158.0, 93.0)
- added REF**125: PinSocket_1x02_P2.54mm_Vertical_SMD_Pin1Right, Connector_PinSocket_2.54mm:PinSocket_1x02_P2.54mm_Vertical_SMD_Pin1Right, F.Cu at (158.0, 82.8)
- added REF**126: PinSocket_1x02_P2.54mm_Vertical_SMD_Pin1Right, Connector_PinSocket_2.54mm:PinSocket_1x02_P2.54mm_Vertical_SMD_Pin1Right, F.Cu at (173.0, 75.0)
- added REF**127: R_1206_3216Metric_Pad1.30x1.75mm_HandSolder, Resistor_SMD:R_1206_3216Metric_Pad1.30x1.75mm_HandSolder, B.Cu at (173.0, 67.0)
- added REF**128: PinSocket_1x03_P2.54mm_Vertical, Connector_PinSocket_2.54mm:PinSocket_1x03_P2.54mm_Vertical, F.Cu at (173.0, 57.5)
- added REF**129: R_1206_3216Metric_Pad1.30x1.75mm_HandSolder, Resistor_SMD:R_1206_3216Metric_Pad1.30x1.75mm_HandSolder, B.Cu at (173.0, 53.0)
- added REF**130: PinSocket_1x02_P2.54mm_Vertical_SMD_Pin1Right, Connector_PinSocket_2.54mm:PinSocket_1x02_P2.54mm_Vertical_SMD_Pin1Right, F.Cu at (173.0, 42.8)
- added REF**131: PinSocket_1x02_P2.54mm_Vertical_SMD_Pin1Right, Connector_PinSocket_2.54mm:PinSocket_1x02_P2.54mm_Vertical_SMD_Pin1Right, F.Cu at (168.0, 115.0)
- added REF**132: R_1206_3216Metric_Pad1.30x1.75mm_HandSolder, Resistor_SMD:R_1206_3216Metric_Pad1.30x1.75mm_HandSolder, B.Cu at (168.0, 107.0)
- added REF**133: PinSocket_1x03_P2.54mm_Vertical, Connector_PinSocket_2.54mm:PinSocket_1x03_P2.54mm_Vertical, F.Cu at (168.0, 97.5)
- added REF**134: R_1206_3216Metric_Pad1.30x1.75mm_HandSolder, Resistor_SMD:R_1206_3216Metric_Pad1.30x1.75mm_HandSolder, B.Cu at (168.0, 93.0)
- added REF**135: PinSocket_1x02_P2.54mm_Vertical_SMD_Pin1Right, Connector_PinSocket_2.54mm:PinSocket_1x02_P2.54mm_Vertical_SMD_Pin1Right, F.Cu at (168.0, 82.8)
- added REF**136: PinSocket_1x02_P2.54mm_Vertical_SMD_Pin1Right, Connector_PinSocket_2.54mm:PinSocket_1x02_P2.54mm_Vertical_SMD_Pin1Right, F.Cu at (183.0, 75.0)
- added REF**137: R_1206_3216Metric_Pad1.30x1.75mm_HandSolder, Resistor_SMD:R_1206_3216Metric_Pad1.30x1.75mm_HandSolder, B.Cu at (183.0, 67.0)
- added REF**138: PinSocket_1x03_P2.54mm_Vertical, Connector_PinSocket_2.54mm:PinSocket_1x03_P2.54mm_Vertical, F.Cu at (183.0, 57.5)
- added REF**139: R_1206_3216Metric_Pad1.30x1.75mm_HandSolder, Resistor_SMD:R_1206_3216Metric_Pad1.30x1.75mm_HandSolder, B.Cu at (183.0, 53.0)
- added REF**140: PinSocket_1x02_P2.54mm_Vertical_SMD_Pin1Right, Connector_PinSocket_2.54mm:PinSocket_1x02_P2.54mm_Vertical_SMD_Pin1Right, F.Cu at (183.0, 42.8)
- added REF**141: PinSocket_1x02_P2.54mm_Vertical_SMD_Pin1Right, Connector_PinSocket_2.54mm:PinSocket_1x02_P2.54mm_Vertical_SMD_Pin1Right, F.Cu at (178.0, 115.0)
- added REF**142: R_1206_3216Metric_Pad1.30x1.75mm_HandSolder, Resistor_SMD:R_1206_3216Metric_Pad1.30x1.75mm_HandSolder, B.Cu at (178.0, 107.0)
- added REF**143: PinSocket_1x03_P2.54mm_Vertical, Connector_PinSocket_2.54mm:PinSocket_1x03_P2.54mm_Vertical, F.Cu at (178.0, 97.5)
- added REF**144: R_1206_3216Metric_Pad1.30x1.75mm_HandSolder, Resistor_SMD:R_1206_3216Metric_Pad1.30x1.75mm_HandSolder, B.Cu at (178.0, 93.0)
- added REF**145: PinSocket_1x02_P2.54mm_Vertical_SMD_Pin1Right, Connector_PinSocket_2.54mm:PinSocket_1x02_P2.54mm_Vertical_SMD_Pin1Right, F.Cu at (178.0, 82.8)
- added REF**146: PinSocket_1x02_P2.54mm_Vertical_SMD_Pin1Right, Connector_PinSocket_2.54mm:PinSocket_1x02_P2.54mm_Vertical_SMD_Pin1Right, F.Cu at (193.0, 75.0)
- added REF**147: R_1206_3216Metric_Pad1.30x1.75mm_HandSolder, Resistor_SMD:R_1206_3216Metric_Pad1.30x1.75mm_HandSolder, B.Cu at (193.0, 67.0)
- added REF**148: PinSocket_1x03_P2.54mm_Vertical, Connector_PinSocket_2.54mm:PinSocket_1x03_P2.54mm_Vertical, F.Cu at (193.0, 57.5)
- added REF**149: R_1206_3216Metric_Pad1.30x1.75mm_HandSolder, Resistor_SMD:R_1206_3216Metric_Pad1.30x1.75mm_HandSolder, B.Cu at (193.0, 53.0)
- added REF**150: PinSocket_1x02_P2.54mm_Vertical_SMD_Pin1Right, Connector_PinSocket_2.54mm:PinSocket_1x02_P2.54mm_Vertical_SMD_Pin1Right, F.Cu at (193.0, 42.8)
- added REF**151: PinSocket_1x02_P2.54mm_Vertical_SMD_Pin1Right, Connector_PinSocket_2.54mm:PinSocket_1x02_P2.54mm_Vertical_SMD_Pin1Right, F.Cu at (188.0, 115.0)
- added REF**152: R_1206_3216Metric_Pad1.30x1.75mm_HandSolder, Resistor_SMD:R_1206_3216Metric_Pad1.30x1.75mm_HandSolder, B.Cu at (188.0, 107.0)
- added REF**153: PinSocket_1x03_P2.54mm_Vertical, Connector_PinSocket_2.54mm:PinSocket_1x03_P2.54mm_Vertical, F.Cu at (188.0, 97.5)
- added REF**154: R_1206_3216Metric_Pad1.30x1.75mm_HandSolder, Resistor_SMD:R_1206_3216Metric_Pad1.30x1.75mm_HandSolder, B.Cu at (188.0, 93.0)
- added REF**155: PinSocket_1x02_P2.54mm_Vertical_SMD_Pin1Right, Connector_PinSocket_2.54mm:PinSocket_1x02_P2.54mm_Vertical_SMD_Pin1Right, F.Cu at (188.0, 82.8)
- added REF**161: PinSocket_1x02_P2.54mm_Vertical_SMD_Pin1Right, Connector_PinSocket_2.54mm:PinSocket_1x02_P2.54mm_Vertical_SMD_Pin1Right, F.Cu at (198.0, 115.0)
- added REF**162: R_1206_3216Metric_Pad1.30x1.75mm_HandSolder, Resistor_SMD:R_1206_3216Metric_Pad1.30x1.75mm_HandSolder, B.Cu at (198.0, 107.0)
- added REF**163: PinSocket_1x03_P2.54mm_Vertical, Connector_PinSocket_2.54mm:PinSocket_1x03_P2.54mm_Vertical, F.Cu at (198.0, 97.5)
- added REF**164: R_1206_3216Metric_Pad1.30x1.75mm_HandSolder, Resistor_SMD:R_1206_3216Metric_Pad1.30x1.75mm_HandSolder, B.Cu at (198.0, 93.0)
- added REF**165: PinSocket_1x02_P2.54mm_Vertical_SMD_Pin1Right, Connector_PinSocket_2.54mm:PinSocket_1x02_P2.54mm_Vertical_SMD_Pin1Right, F.Cu at (198.0, 82.8)
- added REF**49: R_1206_3216Metric_Pad1.30x1.75mm_HandSolder, Resistor_SMD:R_1206_3216Metric_Pad1.30x1.75mm_HandSolder, B.Cu at (93.0, 53.0)
- added REF**50: PinSocket_1x02_P2.54mm_Vertical_SMD_Pin1Right, Connector_PinSocket_2.54mm:PinSocket_1x02_P2.54mm_Vertical_SMD_Pin1Right, F.Cu at (93.0, 42.8)
- added REF**51: PinSocket_1x02_P2.54mm_Vertical_SMD_Pin1Right, Connector_PinSocket_2.54mm:PinSocket_1x02_P2.54mm_Vertical_SMD_Pin1Right, F.Cu at (88.0, 115.0)
- added REF**94: R_1206_3216Metric_Pad1.30x1.75mm_HandSolder, Resistor_SMD:R_1206_3216Metric_Pad1.30x1.75mm_HandSolder, B.Cu at (128.0, 93.0)
- added REF**95: PinSocket_1x02_P2.54mm_Vertical_SMD_Pin1Right, Connector_PinSocket_2.54mm:PinSocket_1x02_P2.54mm_Vertical_SMD_Pin1Right, F.Cu at (128.0, 82.8)
- added REF**96: PinSocket_1x02_P2.54mm_Vertical_SMD_Pin1Right, Connector_PinSocket_2.54mm:PinSocket_1x02_P2.54mm_Vertical_SMD_Pin1Right, F.Cu at (143.0, 75.0)
- REF**11, REF**20, REF**26, REF**35, REF**41, REF**5, REF**56, REF**65, REF**71, REF**80, REF**86: value PinSocket_1x03_P2.54mm_Vertical -> PinSocket_1x02_P2.54mm_Vertical_SMD_Pin1Right; footprint Connector_PinSocket_2.54mm:PinSocket_1x03_P2.54mm_Vertical -> Connector_PinSocket_2.54mm:PinSocket_1x02_P2.54mm_Vertical_SMD_Pin1Right
- REF**12, REF**19, REF**22, REF**24, REF**27, REF**34, REF**37, REF**39, REF**4, REF**42, REF**52, REF**54, REF**57, REF**64, REF**67, REF**69, REF**7, REF**72, REF**79, REF**87, REF**9, REF**97, REF**99: value PinSocket_1x02_P2.54mm_Vertical_SMD_Pin1Right -> R_1206_3216Metric_Pad1.30x1.75mm_HandSolder; footprint Connector_PinSocket_2.54mm:PinSocket_1x02_P2.54mm_Vertical_SMD_Pin1Right -> Resistor_SMD:R_1206_3216Metric_Pad1.30x1.75mm_HandSolder; moved to B.Cu
- REF**13, REF**18, REF**28, REF**3, REF**33, REF**43, REF**48, REF**58, REF**63, REF**73, REF**78, REF**88, REF**93: value PinSocket_1x02_P2.54mm_Vertical_SMD_Pin1Right -> PinSocket_1x03_P2.54mm_Vertical; footprint Connector_PinSocket_2.54mm:PinSocket_1x02_P2.54mm_Vertical_SMD_Pin1Right -> Connector_PinSocket_2.54mm:PinSocket_1x03_P2.54mm_Vertical
- REF**14, REF**17, REF**2, REF**29, REF**32, REF**44, REF**47, REF**59, REF**62, REF**74, REF**77, REF**89, REF**92: value PinSocket_1x03_P2.54mm_Vertical -> R_1206_3216Metric_Pad1.30x1.75mm_HandSolder; footprint Connector_PinSocket_2.54mm:PinSocket_1x03_P2.54mm_Vertical -> Resistor_SMD:R_1206_3216Metric_Pad1.30x1.75mm_HandSolder; moved to B.Cu
- moved REF**72 84.6 mm to (108.0, 107.0), turned to -90 degrees
- moved REF**71 79.6 mm to (108.0, 115.0)
- moved REF**79 76.6 mm to (123.0, 53.0), turned to 90 degrees
- moved REF**42 73.1 mm to (78.0, 107.0), turned to -90 degrees
- moved REF**97 73.0 mm to (143.0, 67.0), turned to -90 degrees
- moved REF**80 70.8 mm to (123.0, 42.8)
- moved REF**98 68.0 mm to (143.0, 57.5)
- moved REF**54 67.4 mm to (88.0, 93.0), turned to 90 degrees
- moved REF**41 67.3 mm to (78.0, 115.0)
- moved REF**12 65.9 mm to (48.0, 107.0), turned to -90 degrees
- moved REF**99 62.6 mm to (143.0, 53.0), turned to 90 degrees
- moved REF**88 62.5 mm to (133.0, 57.5)
- moved REF**19 62.2 mm to (63.0, 53.0), turned to 90 degrees
- moved REF**93 61.8 mm to (128.0, 97.5)
- moved REF**92 60.8 mm to (128.0, 107.0), turned to -90 degrees
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Connections:
- REF** pad 1: (no net) -> P.Pos
- REF** pad 3: (no net) -> P.Neg
- REF** pad 4: (no net) -> +12
- REF** pad 9: (no net) -> -12
- REF**10 pad 2: (no net) -> Signal.Ground
- REF**11 pad 2: Power.Ground -> (no net)
- REF**12 pad 1: (no net) -> P.Neg
- REF**12 pad 2: Signal.Ground -> -12
- REF**13 pad 1: (no net) -> P.Pos
- REF**13 pad 2: (no net) -> Power.Ground
- REF**14 pad 1: (no net) -> P.Pos
- REF**14 pad 2: Power.Ground -> +12
- REF**17 pad 1: (no net) -> P.Neg
- REF**17 pad 2: Power.Ground -> -12
- REF**18 pad 1: (no net) -> P.Pos
- REF**18 pad 2: Signal.Ground -> Power.Ground
- REF**19 pad 1: (no net) -> P.Pos
- REF**19 pad 2: (no net) -> +12
- REF**2 pad 1: (no net) -> P.Neg
- REF**2 pad 2: Power.Ground -> -12
- REF**20 pad 2: Power.Ground -> Signal.Ground
- REF**21 pad 2: Signal.Ground -> (no net)
- REF**22 pad 1: (no net) -> P.Neg
- REF**22 pad 2: (no net) -> -12
- REF**23 pad 1: (no net) -> P.Pos
- REF**23 pad 3: (no net) -> P.Neg
- REF**24 pad 1: (no net) -> P.Pos
- REF**24 pad 2: Signal.Ground -> +12
- REF**25 pad 2: (no net) -> Signal.Ground
- REF**26 pad 2: Power.Ground -> (no net)
- REF**27 pad 1: (no net) -> P.Neg
- REF**27 pad 2: Signal.Ground -> -12
- REF**28 pad 1: (no net) -> P.Pos
- REF**28 pad 2: (no net) -> Power.Ground
- REF**29 pad 1: (no net) -> P.Pos
- REF**29 pad 2: Power.Ground -> +12
- REF**3 pad 1: (no net) -> P.Pos
- REF**3 pad 2: Signal.Ground -> Power.Ground
- REF**32 pad 1: (no net) -> P.Neg
- REF**32 pad 2: Power.Ground -> -12
- REF**33 pad 1: (no net) -> P.Pos
- REF**33 pad 2: Signal.Ground -> Power.Ground
- REF**34 pad 1: (no net) -> P.Pos
- REF**34 pad 2: (no net) -> +12
- REF**35 pad 2: Power.Ground -> Signal.Ground
- REF**36 pad 2: Signal.Ground -> (no net)
- REF**37 pad 1: (no net) -> P.Neg
- REF**37 pad 2: (no net) -> -12
- REF**38 pad 1: (no net) -> P.Pos
- REF**38 pad 3: (no net) -> P.Neg
- REF**39 pad 1: (no net) -> P.Pos
- REF**39 pad 2: Signal.Ground -> +12
- REF**4 pad 1: (no net) -> P.Pos
- REF**4 pad 2: (no net) -> +12
- REF**40 pad 2: (no net) -> Signal.Ground
- REF**41 pad 2: Power.Ground -> (no net)
- REF**42 pad 1: (no net) -> P.Neg
- REF**42 pad 2: Signal.Ground -> -12
- REF**43 pad 1: (no net) -> P.Pos
- REF**43 pad 2: (no net) -> Power.Ground
- REF**44 pad 1: (no net) -> P.Pos
- REF**44 pad 2: Power.Ground -> +12
- REF**47 pad 1: (no net) -> P.Neg
- REF**47 pad 2: Power.Ground -> -12
- REF**48 pad 1: (no net) -> P.Pos
- REF**48 pad 2: Signal.Ground -> Power.Ground
- REF**5 pad 2: Power.Ground -> Signal.Ground
- REF**52 pad 1: (no net) -> P.Neg
- REF**52 pad 2: (no net) -> -12
- REF**53 pad 1: (no net) -> P.Pos
- REF**53 pad 3: (no net) -> P.Neg
- REF**54 pad 1: (no net) -> P.Pos
- REF**54 pad 2: Signal.Ground -> +12
- REF**55 pad 2: (no net) -> Signal.Ground
- REF**56 pad 2: Power.Ground -> (no net)
- REF**57 pad 1: (no net) -> P.Neg
- REF**57 pad 2: Signal.Ground -> -12
- REF**58 pad 1: (no net) -> P.Pos
- REF**58 pad 2: (no net) -> Power.Ground
- REF**59 pad 1: (no net) -> P.Pos
- REF**59 pad 2: Power.Ground -> +12
- REF**6 pad 2: Signal.Ground -> (no net)
- REF**62 pad 1: (no net) -> P.Neg
- REF**62 pad 2: Power.Ground -> -12
- REF**63 pad 1: (no net) -> P.Pos
- REF**63 pad 2: Signal.Ground -> Power.Ground
- REF**64 pad 1: (no net) -> P.Pos
- REF**64 pad 2: (no net) -> +12
- REF**65 pad 2: Power.Ground -> Signal.Ground
- REF**66 pad 2: Signal.Ground -> (no net)
- REF**67 pad 1: (no net) -> P.Neg
- REF**67 pad 2: (no net) -> -12
- REF**68 pad 1: (no net) -> P.Pos
- REF**68 pad 3: (no net) -> P.Neg
- REF**69 pad 1: (no net) -> P.Pos
- REF**69 pad 2: Signal.Ground -> +12
- REF**7 pad 1: (no net) -> P.Neg
- REF**7 pad 2: (no net) -> -12
- REF**70 pad 2: (no net) -> Signal.Ground
- REF**71 pad 2: Power.Ground -> (no net)
- REF**72 pad 1: (no net) -> P.Neg
- REF**72 pad 2: Signal.Ground -> -12
- REF**73 pad 1: (no net) -> P.Pos
- REF**73 pad 2: (no net) -> Power.Ground
- REF**74 pad 1: (no net) -> P.Pos
- REF**74 pad 2: Power.Ground -> +12
- REF**77 pad 1: (no net) -> P.Neg
- REF**77 pad 2: Power.Ground -> -12
- REF**78 pad 1: (no net) -> P.Pos
- REF**78 pad 2: Signal.Ground -> Power.Ground
- REF**79 pad 1: (no net) -> P.Pos
- REF**79 pad 2: (no net) -> +12
- REF**8 pad 1: (no net) -> P.Pos
- REF**8 pad 3: (no net) -> P.Neg
- REF**80 pad 2: Power.Ground -> Signal.Ground
- REF**86 pad 2: Power.Ground -> (no net)
- REF**87 pad 1: (no net) -> P.Neg
- REF**87 pad 2: Signal.Ground -> -12
- REF**88 pad 1: (no net) -> P.Pos
- REF**88 pad 2: (no net) -> Power.Ground
- REF**89 pad 1: (no net) -> P.Pos
- REF**89 pad 2: Power.Ground -> +12
- REF**9 pad 1: (no net) -> P.Pos
- REF**9 pad 2: Signal.Ground -> +12
- REF**92 pad 1: (no net) -> P.Neg
- REF**92 pad 2: Power.Ground -> -12
- REF**93 pad 1: (no net) -> P.Pos
- REF**93 pad 2: Signal.Ground -> Power.Ground
- REF**97 pad 1: (no net) -> P.Neg
- REF**97 pad 2: (no net) -> -12
- REF**98 pad 1: (no net) -> P.Pos
- REF**98 pad 3: (no net) -> P.Neg
- REF**99 pad 1: (no net) -> P.Pos
- REF**99 pad 2: Signal.Ground -> +12
Routing:
- net +12: track 0.00 -> 448.4 mm
- net -12: track 0.00 -> 442.7 mm
- net P.Neg: track 0.00 -> 93.2 mm
- net P.Pos: track 0.00 -> 93.1 mm
Other:
- board text added: "https://github.com/barajasalfredo13/32.Channel.Amp"
